File: hardware/MilkPompV2.kicad_pcb (KiCad board)
At the start: 2 copper layers, 160 x 67.3 mm, 67 parts, among them J1 OUTPUTS, J2 Conn_Display, J3 Program_Conn, J4 Conn_02x07_Odd_Even, J6 PWR INPUT, K1 G5LE-1, Q1 BC847, Q2 BC847, SW1 SW_IO, SW2 SW_IO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

Commit message: naming is complete
Parts:
- moved F1 1.78 mm to (98.3, 120.6)
Routing:
- net +12V: track 80.2 -> 81.9 mm
- net Net-(D4-Pad2): track 8.73 -> 6.95 mm
Other:
- board text added: "+12V"
- board text added: "+3V3"
- board text added: "BTN_IO"
- board text added: "BTN_MODE"
- board text added: "BTN_START"
- board text added: "Buzzer"
- board text added: "DISPLAY"
- board text added: "Display Connector"
- board text added: "FLOW"
- board text added: "GND"
- board text added: "IN"
- board text added: "Mainboard Connector"
- board text added: "NC"
- board text added: "NO"
- board text added: "Relay"
- board text added: "SWCLK"
- board text added: "SWDIO"
