File: hardware/MilkPompV2.kicad_pcb (KiCad board)
At the start: 2 copper layers, 160 x 67.3 mm, 67 parts, among them J1 OUTPUTS, J2 Conn_Display, J3 Program_Conn, J4 Conn_02x07_Odd_Even, J6 PWR INPUT, K1 G5LE-1, Q1 BC847, Q2 BC847, SW1 SW_IO, SW2 SW_IO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

Commit message: arrangement has been made
Other:
- board text added: "MILKPOMP20221206"
- board text added: "www.eltassan.com Adana/Türkiye Eyüp Karakaya Donanım Tasarım Mühendisi"
- board text removed: "MilkPomp"
