File: hardware/buttons.kicad_sch (KiCad schematic)
At the start: 6 parts, among them SW1 SW_IO, SW2 SW_IO, SW3 SW_IO

Commit message: arrangement has been made
Other:
- company: (none) -> ELTASSAN LTD
- title: (none) -> MILK POMP
Changed lines of the file:
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@@
 (kicad_sch (version 20211123) (generator eeschema)
   (paper "A4")
+  (title_block
+    (title "MILK POMP")
+    (date "2022-12-06")
+    (rev "V2")
+    (company "ELTASSAN LTD")
+    (comment 1 "EYYÜP KARAKAYA ")
+    (comment 2 "DONANIM TASARIM MÜHENDİSİ")
+  )
   (junction (at 168.148 99.06) (diameter 0) (color 0 0 0 0)
   )
