File: hardware/mcu.kicad_sch (KiCad schematic)
At the start: 9 parts, among them J3 Program_Conn, U1 STM32G030F6P6TR

Commit message: arrangement has been made
Other:
- company: (none) -> ELTASSAN LTD
- title: (none) -> MILK POMP
Changed lines of the file:
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@@
 (kicad_sch (version 20211123) (generator eeschema)
   (paper "A4")
+  (title_block
+    (title "MILK POMP")
+    (date "2022-12-06")
+    (rev "V2")
+    (company "ELTASSAN LTD")
+    (comment 1 "EYYÜP KARAKAYA ")
+    (comment 2 "DONANIM TASARIM MÜHENDİSİ")
+  )
   (junction (at 35.179 29.972) (diameter 0) (color 0 0 0 0)
   )
