File: hardware/power.kicad_sch (KiCad schematic)
At the start: 11 parts, among them U4 TPS7A4901DGNT

Commit message: arrangement has been made
Other:
- company: (none) -> ELTASSAN LTD
- title: MilkPompPower -> MILK POMP
Changed lines of the file:
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@@
   (paper "A4")
   (title_block
-    (title "MilkPompPower")
-    (date "2022-12-02")
-    (rev "2.0")
+    (title "MILK POMP")
+    (date "2022-12-06")
+    (rev "V2")
+    (company "ELTASSAN LTD")
+    (comment 1 "EYYÜP KARAKAYA ")
+    (comment 2 "DONANIM TASARIM MÜHENDİSİ")
   )
   (junction (at 203.454 124.714) (diameter 0) (color 0 0 0 0)
