File: hardware/relay.kicad_sch (KiCad schematic)
At the start: 7 parts, among them K1 G5LE-1, Q1 BC847

Commit message: arrangement has been made
Other:
- company: (none) -> ELTASSAN LTD
- title: (none) -> MILK POMP
Changed lines of the file:
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@@
 (kicad_sch (version 20211123) (generator eeschema)
   (paper "A4")
+  (title_block
+    (title "MILK POMP")
+    (date "2022-12-06")
+    (rev "V2")
+    (company "ELTASSAN LTD")
+    (comment 1 "EYYÜP KARAKAYA ")
+    (comment 2 "DONANIM TASARIM MÜHENDİSİ")
+  )
   (junction (at 150.876 67.818) (diameter 0) (color 0 0 0 0)
   )

Commit message: name stardandi added, readme file updated
Parts:
- removed D3: 1N4148, Diode_THT:D_DO-35_SOD27_P7.62mm_Horizontal, symbol Diode:1N4148
- added D3: SBR3A40SAQ, Diode_SMD:D_SMB_Handsoldering, symbol Device:D
Connections:
- net +12V: now also D3.1 (K)
- net at D2.1 (K), K1.2, Q1.3 (C): now also D3.2 (A)
Changed lines of the file:
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@@
     (pin "5")
-  )
-  (symbol (lib_id "Diode:1N4148") (at 150.876 78.74 270) (unit 1)
-    (in_bom yes) (on_board yes)
-    (property "Reference" "D3" (id 0) (at 147.066 76.2 90)
-      (effects (font (size 1.27 1.27)) (justify left))
-    )
-    (property "Value" "1N4148" (id 1) (at 143.256 81.915 90)
-      (effects (font (size 1.27 1.27)) (justify left))
-    )
-    (property "Footprint" "Diode_THT:D_DO-35_SOD27_P7.62mm_Horizontal" (id 2) (at 146.431 78.74 0)
-      (effects (font (size 1.27 1.27)) hide)
-    )
-    (property "Datasheet" "https://assets.nexperia.com/documents/data-sheet/1N4148_1N4448.pdf" (id 3) (at 150.876 78.74 0)
-      (effects (font (size 1.27 1.27)) hide)
-    )
-    (pin "1")
-    (pin "2")
   )
   (symbol (lib_id "power:GND") (at 161.798 106.68 0) (unit 1)
@@
       (effects (font (size 1.27 1.27)) hide)
     )
+    (pin "1")
+    (pin "2")
+  )
+  (symbol (lib_id "Device:D") (at 150.876 78.74 270) (unit 1)
+    (in_bom yes) (on_board yes)
+    (property "Reference" "D3" (id 0) (at 148.336 78.74 0))
+    (property "Value" "SBR3A40SAQ" (id 1) (at 153.416 77.47 0))
+    (property "Footprint" "Diode_SMD:D_SMB_Handsoldering" (id 2) (at 150.876 78.74 0)
+      (effects (font (size 1.27 1.27)) hide)
+    )
+    (property "Datasheet" "https://www.diodes.com/assets/Datasheets/SBR3A40SA.pdf" (id 3) (at 150.876 78.74 0)
+      (effects (font (size 1.27 1.27)) hide)
+    )
+    (property "DIGIKEY_PART_NUMBER" "SBR3A40SAQ-13DICT-ND" (id 4) (at 150.876 78.74 0)
+      (effects (font (size 1.27 1.27)) hide)
+    )
+    (property "Digikey" "SBR3A40SAQ-13DICT-ND" (id 5) (at 150.876 78.74 0)
+      (effects (font (size 1.27 1.27)) hide)
+    )
